Commit message: Made jnts more damp stiff & fixed jnt for easy sim

File: cobot-description/urdf/ag95/ag95.transmission.xacro (robot description, xacro)
@@ -11,5 +11,5 @@
         </actuator>
     </transmission>
-    <gazebo>
+    <!-- <gazebo>
         <plugin filename="libroboticsgroup_upatras_gazebo_mimic_joint_plugin.so" name="mimic_finger2">
           <joint>gripper_finger1_joint</joint>
@@ -52,5 +52,5 @@
           <multiplier>1.49462955</multiplier>
         </plugin>
-    </gazebo>
+    </gazebo> -->
   </xacro:macro>
 </robot>

File: cobot-description/urdf/ag95/ag95.xacro (robot description, xacro)
@@ -1,2 +1,3 @@
+<?xml version="1.0"?>
 <robot xmlns:xacro="http://wiki.ros.org/xacro">
 	<xacro:macro name="ag95" params="joint_origin_offset joint_origin_angle hw_interface gripper_parent">
@@ -25,33 +26,41 @@
 		</link>
 		<gazebo reference="gripper_base_link">
+			<mu1>
+				100000
+			</mu1>
+			<mu2>
+				100000
+			</mu2>
+			<kp>
+				100000000.0
+			</kp>
+			<kd>
+				10.0
+			</kd>
+			<maxVel>
+				0.0
+			</maxVel>
+		</gazebo>
+		<joint name="gripper_finger1_joint" type="revolute">
+			<parent link="gripper_base_link" />
+			<child link="gripper_finger1_knuckle_link" />
+			<axis xyz="0 -1 0" />
+			<origin rpy="0.0 0.0 3.14159265359" xyz="-0.016 0 0.10586" />
+			<limit effort="0.0001" lower="0.0" upper="0.65" velocity="0.0" />
+		</joint>
+		<gazebo reference="gripper_finger1_joint">
 			<implicitSpringDamper>
 				1
 			</implicitSpringDamper>
-			<mu1>
-				100000
-			</mu1>
-			<mu2>
-				100000
-			</mu2>
-			<kp>
-				100000000.0
-			</kp>
-			<kd>
-				1.0
-			</kd>
-		</gazebo>
-		<joint name="gripper_finger1_joint" type="revolute">
-			<parent link="gripper_base_link" />
-			<child link="gripper_finger1_knuckle_link" />
-			<axis xyz="0 -1 0" />
-			<origin rpy="0.0 0.0 3.14159265359" xyz="-0.016 0 0.10586" />
-			<limit effort="1000" lower="0.0" upper="0.65" velocity="2.0" />
-		</joint>
-		<joint name="gripper_finger2_joint" type="revolute">
+			<springStiffness>
+				2000000
+			</springStiffness>
+		</gazebo>
+		<joint name="gripper_finger2_joint" type="fixed">
 			<parent link="gripper_base_link" />
 			<child link="gripper_finger2_knuckle_link" />
 			<axis xyz="0 -1 0" />
 			<origin rpy="0.0 0.0 0.0" xyz="0.0160 0 0.10586" />
-			<limit effort="1000" lower="-3.14" upper="3.14" velocity="100.0" />
+			<limit effort="0.0001" lower="-3.14" upper="3.14" velocity="0.0" />
 			<mimic joint="gripper_finger1_joint" />
 		</joint>
@@ -74,19 +83,19 @@
 		</link>
 		<gazebo reference="gripper_finger1_knuckle_link">
-			<implicitSpringDamper>
-				1
-			</implicitSpringDamper>
-			<mu1>
-				100000
-			</mu1>
-			<mu2>
-				100000
-			</mu2>
-			<kp>
-				100000000.0
-			</kp>
-			<kd>
-				1.0
-			</kd>
+			<mu1>
+				100000
+			</mu1>
+			<mu2>
+				100000
+			</mu2>
+			<kp>
+				100000000.0
+			</kp>
+			<kd>
+				10.0
+			</kd>
+			<maxVel>
+				0.0
+			</maxVel>
 		</gazebo>
 		<link name="gripper_finger2_knuckle_link">
@@ -108,34 +117,34 @@
 		</link>
 		<gazebo reference="gripper_finger2_knuckle_link">
-			<implicitSpringDamper>
-				1
-			</implicitSpringDamper>
-			<mu1>
-				100000
-			</mu1>
-			<mu2>
-				100000
-			</mu2>
-			<kp>
-				100000000.0
-			</kp>
-			<kd>
-				1.0
-			</kd>
-		</gazebo>
-		<joint name="gripper_finger1_finger_joint" type="continuous">
+			<mu1>
+				100000
+			</mu1>
+			<mu2>
+				100000
+			</mu2>
+			<kp>
+				100000000.0
+			</kp>
+			<kd>
+				10.0
+			</kd>
+			<maxVel>
+				0.0
+			</maxVel>
+		</gazebo>
+		<joint name="gripper_finger1_finger_joint" type="fixed">
 			<parent link="gripper_finger1_knuckle_link" />
 			<child link="gripper_finger1_finger_link" />
 			<axis xyz="0 -1 0" />
 			<origin rpy="0 0 0" xyz="0.0292080077784 0.0 -0.0227132622407" />
-			<limit effort="0.1" lower="-3.14" upper="3.14" velocity="100.0" />
+			<limit effort="0.1" lower="-3.14" upper="3.14" velocity="0.0" />
 			<mimic joint="gripper_finger1_joint" multiplier="0.4563942" offset="0" />
 		</joint>
-		<joint name="gripper_finger2_finger_joint" type="continuous">
+		<joint name="gripper_finger2_finger_joint" type="fixed">
 			<parent link="gripper_finger2_knuckle_link" />
 			<child link="gripper_finger2_finger_link" />
 			<axis xyz="0 -1 0" />
 			<origin rpy="0 0 0" xyz="0.0292080077784 0.0 -0.0227132622407" />
-			<limit effort="0.1" lower="-3.14" upper="3.14" velocity="100.0" />
+			<limit effort="0.1" lower="-3.14" upper="3.14" velocity="0.0" />
 			<mimic joint="gripper_finger1_joint" multiplier="0.4563942" offset="0" />
 		</joint>
@@ -158,19 +167,19 @@
 		</link>
 		<gazebo reference="gripper_finger1_finger_link">
-			<implicitSpringDamper>
-				1
-			</implicitSpringDamper>
-			<mu1>
-				100000
-			</mu1>
-			<mu2>
-				100000
-			</mu2>
-			<kp>
-				100000000.0
-			</kp>
-			<kd>
-				1.0
-			</kd>
+			<mu1>
+				100000
+			</mu1>
+			<mu2>
+				100000
+			</mu2>
+			<kp>
+				100000000.0
+			</kp>
+			<kd>
+				10.0
+			</kd>
+			<maxVel>
+				0.0
+			</maxVel>
 		</gazebo>
 		<link name="gripper_finger2_finger_link">
@@ -192,34 +201,34 @@
 		</link>
 		<gazebo reference="gripper_finger2_finger_link">
-			<implicitSpringDamper>
-				1
-			</implicitSpringDamper>
-			<mu1>
-				100000
-			</mu1>
-			<mu2>
-				100000
-			</mu2>
-			<kp>
-				100000000.0
-			</kp>
-			<kd>
-				1.0
-			</kd>
-		</gazebo>
-		<joint name="gripper_finger1_inner_knuckle_joint" type="continuous">
+			<mu1>
+				100000
+			</mu1>
+			<mu2>
+				100000
+			</mu2>
+			<kp>
+				100000000.0
+			</kp>
+			<kd>
+				10.0
+			</kd>
+			<maxVel>
+				0.0
+			</maxVel>
+		</gazebo>
+		<joint name="gripper_finger1_inner_knuckle_joint" type="fixed">
 			<parent link="gripper_base_link" />
 			<child link="gripper_finger1_inner_knuckle_link" />
 			<axis xyz="0 -1 0" />
 			<origin rpy="0.0 0.0 3.14159265359" xyz="-0.016 0 0.10586" />
-			<limit effort="0.1" lower="-3.14" upper="3.14" velocity="100.0" />
+			<limit effort="0.1" lower="-3.14" upper="3.14" velocity="0.0" />
 			<mimic joint="gripper_finger1_joint" multiplier="1.49462955" offset="0" />
 		</joint>
-		<joint name="gripper_finger2_inner_knuckle_joint" type="continuous">
+		<joint name="gripper_finger2_inner_knuckle_joint" type="fixed">
 			<parent link="gripper_base_link" />
 			<child link="gripper_finger2_inner_knuckle_link" />
 			<axis xyz="0 -1 0" />
 			<origin rpy="0.0 0.0 0.0" xyz="0.016 0 0.10586" />
-			<limit effort="0.1" lower="-3.14" upper="3.14" velocity="100.0" />
+			<limit effort="0.1" lower="-3.14" upper="3.14" velocity="0.0" />
 			<mimic joint="gripper_finger1_joint" multiplier="1.49462955" offset="0" />
 		</joint>
@@ -242,19 +251,19 @@
 		</link>
 		<gazebo reference="gripper_finger1_inner_knuckle_link">
-			<implicitSpringDamper>
-				1
-			</implicitSpringDamper>
-			<mu1>
-				100000
-			</mu1>
-			<mu2>
-				100000
-			</mu2>
-			<kp>
-				100000000.0
-			</kp>
-			<kd>
-				1.0
-			</kd>
+			<mu1>
+				100000
+			</mu1>
+			<mu2>
+				100000
+			</mu2>
+			<kp>
+				100000000.0
+			</kp>
+			<kd>
+				10.0
+			</kd>
+			<maxVel>
+				0.0
+			</maxVel>
 		</gazebo>
 		<link name="gripper_finger2_inner_knuckle_link">
@@ -276,34 +285,34 @@
 		</link>
 		<gazebo reference="gripper_finger2_inner_knuckle_link">
-			<implicitSpringDamper>
-				1
-			</implicitSpringDamper>
-			<mu1>
-				100000
-			</mu1>
-			<mu2>
-				100000
-			</mu2>
-			<kp>
-				100000000.0
-			</kp>
-			<kd>
-				1.0
-			</kd>
-		</gazebo>
-		<joint name="gripper_finger1_finger_tip_joint" type="continuous">
+			<mu1>
+				100000
+			</mu1>
+			<mu2>
+				100000
+			</mu2>
+			<kp>
+				100000000.0
+			</kp>
+			<kd>
+				10.0
+			</kd>
+			<maxVel>
+				0.0
+			</maxVel>
+		</gazebo>
+		<joint name="gripper_finger1_finger_tip_joint" type="fixed">
 			<parent link="gripper_finger1_inner_knuckle_link" />
 			<child link="gripper_finger1_finger_tip_link" />
 			<axis xyz="0 1 0" />
 			<origin rpy="0.0 0.0 0.0" xyz="0.0394969463769 0.0 0.0382752038125 " />
-			<limit effort="0.1" lower="-3.14" upper="3.14" velocity="100.0" />
+			<limit effort="0.1" lower="-3.14" upper="3.14" velocity="0.0" />
 			<mimic joint="gripper_finger1_joint" multiplier="1.49462955" />
 		</joint>
-		<joint name="gripper_finger2_finger_tip_joint" type="continuous">
+		<joint name="gripper_finger2_finger_tip_joint" type="fixed">
 			<parent link="gripper_finger2_inner_knuckle_link" />
 			<child link="gripper_finger2_finger_tip_link" />
 			<axis xyz="0 1 0" />
 			<origin rpy="0.0 0.0 0.0" xyz="0.0394969463769  0.0 0.0382752038125" />
-			<limit effort="0.1" lower="-3.14" upper="3.14" velocity="100.0" />
+			<limit effort="0.1" lower="-3.14" upper="3.14" velocity="0.0" />
 			<mimic joint="gripper_finger1_joint" multiplier="1.49462955" />
 		</joint>
@@ -326,19 +335,19 @@
 		</link>
 		<gazebo reference="gripper_finger1_finger_tip_link">
-			<implicitSpringDamper>
-				1
-			</implicitSpringDamper>
-			<mu1>
-				100000
-			</mu1>
-			<mu2>
-				100000
-			</mu2>
-			<kp>
-				100000000.0
-			</kp>
-			<kd>
-				1.0
-			</kd>
+			<mu1>
+				100000
+			</mu1>
+			<mu2>
+				100000
+			</mu2>
+			<kp>
+				100000000.0
+			</kp>
+			<kd>
+				10.0
+			</kd>
+			<maxVel>
+				0.0
+			</maxVel>
 		</gazebo>
 		<link name="gripper_finger2_finger_tip_link">
@@ -360,19 +369,19 @@
 		</link>
 		<gazebo reference="gripper_finger2_finger_tip_link">
-			<implicitSpringDamper>
-				1
-			</implicitSpringDamper>
-			<mu1>
-				100000
-			</mu1>
-			<mu2>
-				100000
-			</mu2>
-			<kp>
-				100000000.0
-			</kp>
-			<kd>
-				1.0
-			</kd>
+			<mu1>
+				100000
+			</mu1>
+			<mu2>
+				100000
+			</mu2>
+			<kp>
+				100000000.0
+			</kp>
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