Commit message: removed gripper control

File: cobot-description/urdf/ag95/ag95.xacro (robot description, xacro)
@@ -63,5 +63,5 @@
 			<origin rpy="0.0 0.0 0.0" xyz="0.0160 0 0.10586" />
 			<limit effort="0.0001" lower="-3.14" upper="3.14" velocity="0.0" />
-			<mimic joint="gripper_finger1_joint" />
+			<!-- <mimic joint="gripper_finger1_joint" /> -->
 		</joint>
 		<link name="gripper_finger1_knuckle_link">
@@ -139,5 +139,5 @@
 			<origin rpy="0 0 0" xyz="0.0292080077784 0.0 -0.0227132622407" />
 			<limit effort="0.1" lower="-3.14" upper="3.14" velocity="0.0" />
-			<mimic joint="gripper_finger1_joint" multiplier="0.4563942" offset="0" />
+			<!-- <mimic joint="gripper_finger1_joint" multiplier="0.4563942" offset="0" /> -->
 		</joint>
 		<joint name="gripper_finger2_finger_joint" type="fixed">
@@ -147,5 +147,5 @@
 			<origin rpy="0 0 0" xyz="0.0292080077784 0.0 -0.0227132622407" />
 			<limit effort="0.1" lower="-3.14" upper="3.14" velocity="0.0" />
-			<mimic joint="gripper_finger1_joint" multiplier="0.4563942" offset="0" />
+			<!-- <mimic joint="gripper_finger1_joint" multiplier="0.4563942" offset="0" /> -->
 		</joint>
 		<link name="gripper_finger1_finger_link">
@@ -223,5 +223,5 @@
 			<origin rpy="0.0 0.0 3.14159265359" xyz="-0.016 0 0.10586" />
 			<limit effort="0.1" lower="-3.14" upper="3.14" velocity="0.0" />
-			<mimic joint="gripper_finger1_joint" multiplier="1.49462955" offset="0" />
+			<!-- <mimic joint="gripper_finger1_joint" multiplier="1.49462955" offset="0" /> -->
 		</joint>
 		<joint name="gripper_finger2_inner_knuckle_joint" type="fixed">
@@ -231,5 +231,5 @@
 			<origin rpy="0.0 0.0 0.0" xyz="0.016 0 0.10586" />
 			<limit effort="0.1" lower="-3.14" upper="3.14" velocity="0.0" />
-			<mimic joint="gripper_finger1_joint" multiplier="1.49462955" offset="0" />
+			<!-- <mimic joint="gripper_finger1_joint" multiplier="1.49462955" offset="0" /> -->
 		</joint>
 		<link name="gripper_finger1_inner_knuckle_link">
@@ -307,5 +307,5 @@
 			<origin rpy="0.0 0.0 0.0" xyz="0.0394969463769 0.0 0.0382752038125 " />
 			<limit effort="0.1" lower="-3.14" upper="3.14" velocity="0.0" />
-			<mimic joint="gripper_finger1_joint" multiplier="1.49462955" />
+			<!-- <mimic joint="gripper_finger1_joint" multiplier="1.49462955" /> -->
 		</joint>
 		<joint name="gripper_finger2_finger_tip_joint" type="fixed">
@@ -315,5 +315,5 @@
 			<origin rpy="0.0 0.0 0.0" xyz="0.0394969463769  0.0 0.0382752038125" />
 			<limit effort="0.1" lower="-3.14" upper="3.14" velocity="0.0" />
-			<mimic joint="gripper_finger1_joint" multiplier="1.49462955" />
+			<!-- <mimic joint="gripper_finger1_joint" multiplier="1.49462955" /> -->
 		</joint>
 		<link name="gripper_finger1_finger_tip_link">

Commit message: changed colors

File: cobot-description/urdf/ag95/ag95.xacro (robot description, xacro)
@@ -26,4 +26,7 @@
 		</link>
 		<gazebo reference="gripper_base_link">
+			<material>
+				Gazebo/Black
+			</material>
 			<mu1>
 				100000
@@ -83,4 +86,7 @@
 		</link>
 		<gazebo reference="gripper_finger1_knuckle_link">
+			<material>
+				Gazebo/DarkGrey
+			</material>
 			<mu1>
 				100000
@@ -117,4 +123,7 @@
 		</link>
 		<gazebo reference="gripper_finger2_knuckle_link">
+			<material>
+				Gazebo/DarkGrey
+			</material>
 			<mu1>
 				100000
@@ -167,4 +176,7 @@
 		</link>
 		<gazebo reference="gripper_finger1_finger_link">
+			<material>
+				Gazebo/Grey
+			</material>
 			<mu1>
 				100000
@@ -201,4 +213,7 @@
 		</link>
 		<gazebo reference="gripper_finger2_finger_link">
+			<material>
+				Gazebo/Grey
+			</material>
 			<mu1>
 				100000
@@ -251,4 +266,7 @@
 		</link>
 		<gazebo reference="gripper_finger1_inner_knuckle_link">
+			<material>
+				Gazebo/DarkGrey
+			</material>
 			<mu1>
 				100000
@@ -285,4 +303,7 @@
 		</link>
 		<gazebo reference="gripper_finger2_inner_knuckle_link">
+			<material>
+				Gazebo/DarkGrey
+			</material>
 			<mu1>
 				100000
@@ -335,4 +356,7 @@
 		</link>
 		<gazebo reference="gripper_finger1_finger_tip_link">
+			<material>
+				Gazebo/Grey
+			</material>
 			<mu1>
 				100000
@@ -369,4 +393,7 @@
 		</link>
 		<gazebo reference="gripper_finger2_finger_tip_link">
+			<material>
+				Gazebo/Grey
+			</material>
 			<mu1>
 				100000

File: cobot-description/urdf/camera/camera.xacro (robot description, xacro)
@@ -1,2 +1,3 @@
+<?xml version="1.0"?>
 <robot xmlns:xacro="http://wiki.ros.org/xacro">
   <xacro:macro name="camera" params="origin_offset origin_angle camera_parent">
@@ -23,4 +24,7 @@
     </link>
     <gazebo reference="camera_mount_link">
+      <material>
+				Gazebo/Black
+			</material>
       <implicitSpringDamper>1</implicitSpringDamper>
       <mu1>100000</mu1>
