Commit message: Added human_drone model; Renamed industry.world to e_waste.world

File: cobot-env/urdf/e-waste.colors.xacro (robot description, xacro)
@@ -74,5 +74,5 @@
   </gazebo>
   <gazebo reference="toolkit">
-    <material> Gazebo/Orange </material>
+    <material> Gazebo/Purple </material>
   </gazebo>
   <gazebo>
