Commit message: Removed collission mesh for sim

File: cobot-env/urdf/e-waste-setup.xacro (robot description, xacro)
@@ -366,5 +366,5 @@
       xyz="0 0 0" />
   </joint>
-  <link
+  <!-- <link
     name="eth1">
     <inertial>
@@ -418,5 +418,5 @@
     <axis
       xyz="0 0 0" />
-  </joint>
+  </joint> -->
   <link
     name="rpi1">
@@ -1108,5 +1108,5 @@
       xyz="0 0 0" />
   </joint>
-  <link
+  <!-- <link
     name="eth2">
     <inertial>
@@ -1213,5 +1213,5 @@
     <axis
       xyz="0 0 0" />
-  </joint>
+  </joint> -->
   <link
     name="lipo2">
@@ -1267,5 +1267,5 @@
       xyz="0 0 0" />
   </joint>
-  <link
+  <!-- <link
     name="toolkit">
     <inertial>
@@ -1319,5 +1319,5 @@
     <axis
       xyz="0 0 0" />
-  </joint>
+  </joint> -->
   <xacro:include filename="$(find cobot-env)/urdf/e-waste.colors.xacro" />
 </robot>

File: cobot-env/urdf/e-waste.colors.xacro (robot description, xacro)
@@ -25,5 +25,5 @@
     <material> Gazebo/Turquoise </material>
   </gazebo>
-  <gazebo reference="eth1">
+  <!-- <gazebo reference="eth1">
     <material> Gazebo/DarkGrey </material>
   </gazebo>
@@ -33,5 +33,5 @@
   <gazebo reference="eth3">
     <material> Gazebo/DarkGrey </material>
-  </gazebo>
+  </gazebo> -->
   <gazebo reference="rpi1">
     <material> Gazebo/SkyBlue </material>
@@ -73,7 +73,7 @@
     <material> Gazebo/Grey </material>
   </gazebo>
-  <gazebo reference="toolkit">
+  <!-- <gazebo reference="toolkit">
     <material> Gazebo/Purple </material>
-  </gazebo>
+  </gazebo> -->
   <gazebo>
     <static> 1 </static>

Commit message: Updated dev-sim-ctrl for plotting

File: cobot-env/urdf/e-waste-setup.xacro (robot description, xacro)
@@ -366,5 +366,5 @@
       xyz="0 0 0" />
   </joint>
-  <!-- <link
+  <link
     name="eth1">
     <inertial>
@@ -418,5 +418,5 @@
     <axis
       xyz="0 0 0" />
-  </joint> -->
+  </joint>
   <link
     name="rpi1">
@@ -1108,5 +1108,5 @@
       xyz="0 0 0" />
   </joint>
-  <!-- <link
+  <link
     name="eth2">
     <inertial>
@@ -1213,5 +1213,5 @@
     <axis
       xyz="0 0 0" />
-  </joint> -->
+  </joint>
   <link
     name="lipo2">
@@ -1267,5 +1267,5 @@
       xyz="0 0 0" />
   </joint>
-  <!-- <link
+  <link
     name="toolkit">
     <inertial>
@@ -1319,5 +1319,5 @@
     <axis
       xyz="0 0 0" />
-  </joint> -->
+  </joint>
   <xacro:include filename="$(find cobot-env)/urdf/e-waste.colors.xacro" />
 </robot>

File: cobot-env/urdf/e-waste.colors.xacro (robot description, xacro)
@@ -25,5 +25,5 @@
     <material> Gazebo/Turquoise </material>
   </gazebo>
-  <!-- <gazebo reference="eth1">
+  <gazebo reference="eth1">
     <material> Gazebo/DarkGrey </material>
   </gazebo>
@@ -33,5 +33,5 @@
   <gazebo reference="eth3">
     <material> Gazebo/DarkGrey </material>
-  </gazebo> -->
+  </gazebo>
   <gazebo reference="rpi1">
     <material> Gazebo/SkyBlue </material>
@@ -73,7 +73,7 @@
     <material> Gazebo/Grey </material>
   </gazebo>
-  <!-- <gazebo reference="toolkit">
+  <gazebo reference="toolkit">
     <material> Gazebo/Purple </material>
-  </gazebo> -->
+  </gazebo>
   <gazebo>
     <static> 1 </static>

File: cobot-env/urdf/human_drone.xacro (robot description, xacro)
@@ -38,4 +38,12 @@
   <gazebo reference="hd_base_link">
     <material> Gazebo/Orange </material>
+    <collision>
+        <surface>
+          <contact>
+            <collide_without_contact>true</collide_without_contact>
+          </contact>
+        </surface>
+      </collision>
+    <selfCollide>true</selfCollide>
   </gazebo>
 </robot>
