Commit message: Added TCP
Modified files to incorporate TCP

File: cobot-description/urdf/ur5.xacro (robot description, xacro)
@@ -11,4 +11,11 @@
             origin_offset="-0.04 0.04 0"
             origin_angle="0.0 ${-pi/2} ${pi}"/>
+  <!-- Adding TCP -->
+  <joint name='tcp_fixed' type='fixed'>
+    <origin xyz = '0 0 0.182' rpy = '0 0 0'/>
+    <parent link="tool0"/>
+    <child link="tcp"/>
+  </joint>
+  <link name = 'tcp'/>
   <!-- ag95 gripper  -->
   <xacro:include filename="$(find cobot-description)/urdf/ag95/ag95.xacro" />

Commit message: Reverted to usage of realsense via pyrealsense lib
Also changed the TCP offset to 205 mm from tool0 frame.

File: cobot-description/urdf/ur5.xacro (robot description, xacro)
@@ -13,5 +13,5 @@
   <!-- Adding TCP -->
   <joint name='tcp_fixed' type='fixed'>
-    <origin xyz = '0 0 0.182' rpy = '0 0 0'/>
+    <origin xyz = '0 0 0.205' rpy = '0 0 0'/>
     <parent link="tool0"/>
     <child link="tcp"/>

Commit message: Added detailed docs; impl. ur_collision detection ros node;
Removed additional dependencies written in CMakeLists and package

File: cobot-description/urdf/ur5.xacro (robot description, xacro)
@@ -36,3 +36,12 @@
 			<origin rpy="0.0 0.0 0.0" xyz="0 0 0" />
 	</joint>
+  <gazebo reference="shoulder_link">
+    <sensor name='plugin' type='contact'>
+        <contact>
+          <collision>
+            shoulder_link_collision
+          </collision>
+        </contact>
+      </sensor>
+  </gazebo>
 </robot>

File: cobot-env/urdf/human_drone.xacro (robot description, xacro)
@@ -39,4 +39,3 @@
     <material> Gazebo/Orange </material>
   </gazebo>
-  <xacro:include filename="$(find cobot-env)/urdf/human_drone_sensors.xacro"/>
 </robot>
