Commit message: Simulation-e-waste

File: cobot-description/urdf/ur5.urdf (robot description, URDF)
Before this commit: robot ur5_robot, 23 links, 22 joints
Joints:
- joint gripper_finger1_finger_joint: limit lower=-3.14 upper=3.14 effort=0.1 velocity=100.0 -> lower=-3.14 upper=3.14 effort=0.1 velocity=0.0; mimic joint=gripper_finger1_joint multiplier=0.4563942 offset=0 -> (none); type continuous -> fixed
- joint gripper_finger1_finger_tip_joint: limit lower=-3.14 upper=3.14 effort=0.1 velocity=100.0 -> lower=-3.14 upper=3.14 effort=0.1 velocity=0.0; mimic joint=gripper_finger1_joint multiplier=1.49462955 -> (none); type continuous -> fixed
- joint gripper_finger1_inner_knuckle_joint: limit lower=-3.14 upper=3.14 effort=0.1 velocity=100.0 -> lower=-3.14 upper=3.14 effort=0.1 velocity=0.0; mimic joint=gripper_finger1_joint multiplier=1.49462955 offset=0 -> (none); type continuous -> fixed
- joint gripper_finger1_joint: limit lower=0.0 upper=0.65 effort=1000 velocity=2.0 -> lower=0.0 upper=0.65 effort=0.0001 velocity=0.0
- joint gripper_finger2_finger_joint: limit lower=-3.14 upper=3.14 effort=0.1 velocity=100.0 -> lower=-3.14 upper=3.14 effort=0.1 velocity=0.0; mimic joint=gripper_finger1_joint multiplier=0.4563942 offset=0 -> (none); type continuous -> fixed
- joint gripper_finger2_finger_tip_joint: limit lower=-3.14 upper=3.14 effort=0.1 velocity=100.0 -> lower=-3.14 upper=3.14 effort=0.1 velocity=0.0; mimic joint=gripper_finger1_joint multiplier=1.49462955 -> (none); type continuous -> fixed
- joint gripper_finger2_inner_knuckle_joint: limit lower=-3.14 upper=3.14 effort=0.1 velocity=100.0 -> lower=-3.14 upper=3.14 effort=0.1 velocity=0.0; mimic joint=gripper_finger1_joint multiplier=1.49462955 offset=0 -> (none); type continuous -> fixed
- joint gripper_finger2_joint: limit lower=-3.14 upper=3.14 effort=1000 velocity=100.0 -> lower=-3.14 upper=3.14 effort=0.0001 velocity=0.0; mimic joint=gripper_finger1_joint -> (none); type revolute -> fixed
- joint tcp_fixed: origin xyz=0 0 0.182 rpy=0 0 0 -> xyz=0 0 0.205 rpy=0 0 0
